Commit message: merged custom drone config to fork

File: rotors_description/urdf/hummingbird.xacro (robot description, xacro)
@@ -22,5 +22,6 @@
   <xacro:property name="rotor_velocity_slowdown_sim" value="10" />
   <xacro:property name="use_mesh_file" value="true" />
-  <xacro:property name="mesh_file" value="package://rotors_description/meshes/hummingbird.dae" />
+  <!-- <xacro:property name="mesh_file" value="package://rotors_description/meshes/hummingbird.dae" /> -->
+  <xacro:property name="mesh_file" value="package://rotors_description/meshes/shafter.dae" />
   <xacro:property name="mass" value="0.68" /> <!-- [kg] -->
   <xacro:property name="body_width" value="0.1" /> <!-- [m] -->

File: rotors_description/urdf/hummingbird_base.xacro (robot description, xacro)
@@ -20,4 +20,5 @@
   <!-- Instantiate hummingbird "mechanics" -->
   <xacro:include filename="$(find rotors_description)/urdf/hummingbird.xacro" />
+  <xacro:include filename="$(find rotors_description)/urdf/sbl.xacro" />
   <!-- Instantiate a controller. -->
   <xacro:controller_plugin_macro namespace="${namespace}" imu_sub_topic="imu" />
@@ -39,3 +40,8 @@
       wait_to_record_bag="$(arg wait_to_record_bag)" />
   </xacro:if>
+  <!-- Add an 0S0-128 lidar -->
+  <xacro:include filename="$(find lidar_description)/urdf/OS0-128.urdf.xacro"/>
+  <xacro:OS0-128 parent="${namespace}/base_link" name="os_sensor" topic="ouster/points" hz="10" lasers="32" samples="440" collision_range="0.3" min_range="0.3" max_range="50.0">
+    <origin xyz="0.0125 0 0.165" rpy="0 0 0" />
+  </xacro:OS0-128>
 </robot>

File: rotors_description/urdf/multirotor_base.xacro (robot description, xacro)
@@ -50,5 +50,5 @@
         <geometry>
           <xacro:if value="${use_mesh_file}">
-            <mesh filename="${mesh_file}" scale="1 1 1" />
+            <mesh filename="${mesh_file}" scale="0.001 0.001 0.001" />
           </xacro:if>
           <xacro:unless value="${use_mesh_file}">
@@ -92,13 +92,4 @@
         <geometry>
           <!-- <cylinder length="0.005" radius="${radius_rotor}"/> --> <!-- [m] -->
-          <xacro:if value="${use_own_mesh}">
-            <mesh filename="${mesh}"
-              scale="1 1 1" />
-          </xacro:if>
-          <xacro:unless value="${use_own_mesh}">
-            <mesh filename="package://rotors_description/meshes/propeller_${direction}.dae"
-              scale="${radius_rotor} ${radius_rotor} ${radius_rotor}" /> <!-- The propeller meshes have a radius of 1m -->
-            <!-- <box size="${2*radius_rotor} 0.01 0.005"/> -->
-          </xacro:unless>
         </geometry>
       </visual>

File: rotors_description/urdf/pelican_base.xacro (robot description, xacro)
@@ -20,4 +20,10 @@
   <!-- Instantiate pelican "mechanics" -->
   <xacro:include filename="$(find rotors_description)/urdf/pelican.xacro" />
+  <!-- <xacro:include filename="$(find realsense2_description)/urdf/_d435.urdf.xacro"/> -->
+  <xacro:include filename="$(find rotors_description)/urdf/rplidar.xacro"/>
+  <xacro:include filename="$(find rotors_description)/urdf/sbl.xacro" />
+  <xacro:sensor_rplidar parent="${namespace}/base_link" topics_ns="${namespace}/rplidar">
+    <origin xyz="0 0 0.2" rpy="0 0 0"/>
+  </xacro:sensor_rplidar>
   <!-- Instantiate a controller. -->
   <xacro:controller_plugin_macro namespace="${namespace}" imu_sub_topic="imu" />
