Commit message: minor changed in xacro

File: rotors_description/urdf/hummingbird_base.xacro (robot description, xacro)
@@ -45,3 +45,10 @@
     <origin xyz="0.0125 0 0.165" rpy="0 0 0" />
   </xacro:OS0-128>
+  <!-- VLP16 -->
+  <!-- <xacro:arg name="gpu" default="false"/> -->
+  <!-- <xacro:property name="gpu" value="$(arg gpu)" /> -->
+  <!-- <xacro:include filename="$(find lidar_description)/urdf/VLP-16.urdf.xacro"/> -->
+  <!-- <xacro:VLP-16 parent="${namespace}/base_link" name="os_sensor" topic="ouster/points" hz="10" samples="440" gpu="$(arg gpu)" collision_range="0.7" min_range="0.7"> -->
+  <!--   <origin xyz="0.0125 0 0.165" rpy="0 0 0" /> -->
+  <!-- </xacro:VLP-16> -->
 </robot>
